File: hardware/project1/project1.kicad_pcb (KiCad board)
At the start: 2 copper layers, 120 x 120 mm, 46 parts, among them Q1 Q_NMOS_GSD, Q2 Q_NMOS_GSD, Q3 Q_NMOS_GSD, Q4 Q_NMOS_GSD, Q5 TEFT4300, Q6 TEFT4300, Q7 TEFT4300, Q9 TEFT4300, SW2 SW_SPDT, SW3 SW_Push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

Commit message: -
Connections:
- net /Left_motor_1 renamed /l_motor1
Changed lines of the file:
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@@
 			(layers "F.Cu" "F.Mask" "F.Paste")
 			(roundrect_rratio 0.25)
-			(net "/Left_motor_1")
+			(net "/l_motor1")
 			(pinfunction "AIN1_21")
 			(pintype "input")
@@
 			(layers "F.Cu" "F.Mask")
 			(roundrect_rratio 0.5)
-			(net "/Left_motor_1")
+			(net "/l_motor1")
 			(pinfunction "GPIO4_6")
 			(pintype "bidirectional")
@@
 			(layers "*.Cu" "*.Mask")
 			(remove_unused_layers no)
-			(net "/Left_motor_1")
+			(net "/l_motor1")
 			(pinfunction "GPIO4_6")
 			(pintype "bidirectional")
@@
 		(width 0.25)
 		(layer "F.Cu")
-		(net "/Left_motor_1")
+		(net "/l_motor1")
 	)
 	(segment
@@
 		(width 0.25)
 		(layer "F.Cu")
-		(net "/Left_motor_1")
+		(net "/l_motor1")
 	)
 	(segment
@@
 		(width 0.25)
 		(layer "F.Cu")
-		(net "/Left_motor_1")
+		(net "/l_motor1")
 	)
 	(segment
@@
 		(width 0.25)
 		(layer "F.Cu")
-		(net "/Left_motor_1")
+		(net "/l_motor1")
 	)
 	(segment
@@
 		(width 0.25)
 		(layer "F.Cu")
-		(net "/Left_motor_1")
+		(net "/l_motor1")
 	)
 	(segment
@@
 		(width 0.25)
 		(layer "F.Cu")
-		(net "/Left_motor_1")
+		(net "/l_motor1")
 	)
 	(segment
@@
 		(width 0.25)
 		(layer "F.Cu")
-		(net "/Left_motor_1")
+		(net "/l_motor1")
 	)
 	(segment
@@
 		(width 0.25)
 		(layer "F.Cu")
-		(net "/Left_motor_1")
+		(net "/l_motor1")
 	)
 	(segment
@@
 		(width 0.25)
 		(layer "F.Cu")
-		(net "/Left_motor_1")
+		(net "/l_motor1")
 	)
 	(segment
@@
 		(width 0.25)
 		(layer "F.Cu")
-		(net "/Left_motor_1")
+		(net "/l_motor1")
 	)
 	(segment
@@
 		(width 0.25)
 		(layer "F.Cu")
-		(net "/Left_motor_1")
+		(net "/l_motor1")
 	)
 	(segment
@@
 		(width 0.25)
 		(layer "F.Cu")
-		(net "/Left_motor_1")
+		(net "/l_motor1")
 	)
 	(segment
@@
 		(width 0.25)
 		(layer "F.Cu")
-		(net "/Left_motor_1")
+		(net "/l_motor1")
 	)
 	(segment
@@
 		(width 0.25)
 		(layer "F.Cu")
-		(net "/Left_motor_1")
+		(net "/l_motor1")
 	)
 	(segment
@@
 		(width 0.25)
 		(layer "F.Cu")
-		(net "/Left_motor_1")
+		(net "/l_motor1")
 	)
 	(segment
@@
 		(width 0.25)
 		(layer "F.Cu")
-		(net "/Left_motor_1")
+		(net "/l_motor1")
 	)
 	(segment
@@
 		(width 0.25)
 		(layer "F.Cu")
-		(net "/Left_motor_1")
+		(net "/l_motor1")
 	)
 	(segment
@@
 		(width 0.25)
 		(layer "F.Cu")
-		(net "/Left_motor_1")
+		(net "/l_motor1")
 	)
 	(segment
@@
 		(width 0.25)
 		(layer "F.Cu")
-		(net "/Left_motor_1")
+		(net "/l_motor1")
 	)
 	(segment
@@
 		(width 0.25)
 		(layer "F.Cu")
-		(net "/Left_motor_1")
+		(net "/l_motor1")
 	)
 	(segment
@@
 		(width 0.25)
 		(layer "F.Cu")
-		(net "/Left_motor_1")
+		(net "/l_motor1")
 	)
 	(segment
@@
 		(width 0.25)
 		(layer "F.Cu")
-		(net "/Left_motor_1")
+		(net "/l_motor1")
 	)
 	(segment
@@
 		(width 0.25)
 		(layer "F.Cu")
-		(net "/Left_motor_1")
+		(net "/l_motor1")
 	)
 	(segment
@@
 		(width 0.25)
 		(layer "F.Cu")
-		(net "/Left_motor_1")
+		(net "/l_motor1")
 	)
 	(segment
@@
 		(width 0.25)
 		(layer "F.Cu")
-		(net "/Left_motor_1")
+		(net "/l_motor1")
 	)
 	(segment
@@
 		(width 0.25)
 		(layer "F.Cu")
-		(net "/Left_motor_1")
+		(net "/l_motor1")
 	)
 	(segment
@@
 		(width 0.25)
 		(layer "F.Cu")
-		(net "/Left_motor_1")
+		(net "/l_motor1")
 	)
 	(segment
@@
 		(width 0.25)
 		(layer "F.Cu")
-		(net "/Left_motor_1")
+		(net "/l_motor1")
 	)
 	(segment
@@
 		(width 0.25)
 		(layer "F.Cu")
-		(net "/Left_motor_1")
+		(net "/l_motor1")
 	)
 	(segment
@@
 		(width 0.25)
 		(layer "F.Cu")
-		(net "/Left_motor_1")
+		(net "/l_motor1")
 	)
 	(segment
@@
 		(width 0.25)
 		(layer "F.Cu")
-		(net "/Left_motor_1")
+		(net "/l_motor1")
 	)
 	(segment
@@
 		(width 0.25)
 		(layer "F.Cu")
-		(net "/Left_motor_1")
+		(net "/l_motor1")
 	)
 	(segment
@@
 		(width 0.25)
 		(layer "F.Cu")
-		(net "/Left_motor_1")
+		(net "/l_motor1")
 	)
 	(segment
@@
 		(width 0.25)
 		(layer "F.Cu")
-		(net "/Left_motor_1")
+		(net "/l_motor1")
 	)
 	(segment
@@
 		(width 0.25)
 		(layer "F.Cu")
-		(net "/Left_motor_1")
+		(net "/l_motor1")
 	)
 	(via
@@
 		(drill 0.3)
 		(layers "F.Cu" "B.Cu")
-		(net "/Left_motor_1")
+		(net "/l_motor1")
 	)
 	(via
@@
 		(drill 0.3)
 		(layers "F.Cu" "B.Cu")
-		(net "/Left_motor_1")
+		(net "/l_motor1")
 	)
 	(segment
@@
 		(width 0.25)
 		(layer "B.Cu")
-		(net "/Left_motor_1")
+		(net "/l_motor1")
 	)
 	(segment
@@
 		(width 0.25)
 		(layer "B.Cu")
-		(net "/Left_motor_1")
+		(net "/l_motor1")
 	)
 	(segment
@@
 		(width 0.25)
 		(layer "B.Cu")
-		(net "/Left_motor_1")
+		(net "/l_motor1")
 	)
 	(segment
@@
 		(width 0.25)
 		(layer "B.Cu")
-		(net "/Left_motor_1")
+		(net "/l_motor1")
 	)
 	(segment
@@
 		(width 0.25)
 		(layer "B.Cu")
-		(net "/Left_motor_1")
+		(net "/l_motor1")
 	)
 	(segment
@@
 		(width 0.25)
 		(layer "B.Cu")
-		(net "/Left_motor_1")
+		(net "/l_motor1")
 	)
 	(segment
@@
 		(width 0.25)
 		(layer "B.Cu")
-		(net "/Left_motor_1")
+		(net "/l_motor1")
 	)
 	(segment
@@
 		(width 0.25)
 		(layer "B.Cu")
-		(net "/Left_motor_1")
+		(net "/l_motor1")
 	)
 	(segment
@@
 		(width 0.25)
 		(layer "B.Cu")
-		(net "/Left_motor_1")
+		(net "/l_motor1")
 	)
 	(segment
@@
 		(width 0.25)
 		(layer "B.Cu")
-		(net "/Left_motor_1")
+		(net "/l_motor1")
 	)
 	(segment
@@
 		(width 0.25)
 		(layer "B.Cu")
-		(net "/Left_motor_1")
+		(net "/l_motor1")
 	)
 	(segment
@@
 		(width 0.25)
 		(layer "B.Cu")
-		(net "/Left_motor_1")
+		(net "/l_motor1")
 	)
 	(segment
@@
 		(width 0.25)
 		(layer "B.Cu")
-		(net "/Left_motor_1")
+		(net "/l_motor1")
 	)
 	(segment
