File: hardware/project1/project1.kicad_sch (KiCad schematic)
At the start: 46 parts, among them Q1 Q_NMOS_GSD, Q2 Q_NMOS_GSD, Q3 Q_NMOS_GSD, Q4 Q_NMOS_GSD, Q5 TEFT4300, Q6 TEFT4300, Q7 TEFT4300, Q9 TEFT4300, SW2 SW_SPDT, SW3 SW_Push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

Commit message: -
Connections:
- net Left_motor_1 renamed l_motor1
Changed lines of the file:
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@@
 		)
 	)
-	(label "Left_motor_1"
+	(label "l_motor1"
 		(at 273.05 64.77 0)
 		(effects
@@
 		)
 	)
-	(label "Left_motor_1"
+	(label "l_motor1"
 		(at 199.39 187.96 0)
 		(effects
